File: Board/usbc.kicad_sch (KiCad schematic)
At the start: 6 parts, among them J1 USB_C_Receptacle_USB2.0_14P, U1 NCP1117-3.3_SOT223

Commit message: Touch-up module schematics
Changed lines of the file:
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@@
     (effects (font (size 1.27 1.27)) (justify left bottom))
   )
-  (text "USB-C Recepticle" (at 124.46 68.58 0)
+  (text "USB-C Recepticle" (at 151.13 121.92 0)
     (effects (font (size 3 3)) (justify left bottom))
   )

Commit message: Added 3d model to ND68-1u-HS-ARGB and linked all parts to footprints
Parts:
- J1: footprint (none) -> ND68:USB_C_Receptacle_GCT_USB4105-GF-A
Changed lines of the file:
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@@
       (effects (font (size 1.27 1.27)) hide)
     )
-    (property "Footprint" "" (at 116.84 93.98 0)
+    (property "Footprint" "ND68:USB_C_Receptacle_GCT_USB4105-GF-A" (at 116.84 93.98 0)
       (effects (font (size 1.27 1.27)) hide)
     )

Commit message: VERY BASIC pcb layout
Connections:
- net at R1.1: now also J1.A5 (CC1); no longer J1.B5 (CC2)
- net at R2.1: now also J1.B5 (CC2); no longer J1.A5 (CC1)
Other:
- moved on the sheet: R1, R2
Changed lines of the file:
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@@
     )
   )
-  (symbol (lib_id "Device:R") (at 137.16 101.6 0) (unit 1)
+  (symbol (lib_id "Device:R") (at 144.78 101.6 0) (unit 1)
     (in_bom yes) (on_board yes) (dnp no)
-    (property "Reference" "R1" (at 138.43 100.33 0)
-      (effects (font (size 1.27 1.27)) (justify left))
-    )
-    (property "Value" "5.1k" (at 138.43 102.87 0)
-      (effects (font (size 1.27 1.27)) (justify left))
-    )
-    (property "Footprint" "Resistor_SMD:R_0603_1608Metric" (at 135.382 101.6 90)
-      (effects (font (size 1.27 1.27)) hide)
-    )
-    (property "Datasheet" "~" (at 137.16 101.6 0)
-      (effects (font (size 1.27 1.27)) hide)
-    )
-    (property "DigiKey" "311-5.10KHRCT-ND" (at 137.16 101.6 0)
+    (property "Reference" "R1" (at 146.05 100.33 0)
+      (effects (font (size 1.27 1.27)) (justify left))
+    )
+    (property "Value" "5.1k" (at 146.05 102.87 0)
+      (effects (font (size 1.27 1.27)) (justify left))
+    )
+    (property "Footprint" "Resistor_SMD:R_0603_1608Metric" (at 143.002 101.6 90)
+      (effects (font (size 1.27 1.27)) hide)
+    )
+    (property "Datasheet" "~" (at 144.78 101.6 0)
+      (effects (font (size 1.27 1.27)) hide)
+    )
+    (property "DigiKey" "311-5.10KHRCT-ND" (at 144.78 101.6 0)
       (effects (font (size 1.27 1.27)) hide)
     )
@@
     )
   )
-  (symbol (lib_id "Device:R") (at 144.78 101.6 0) (unit 1)
-    (in_bom yes) (on_board yes) (dnp no) (fields_autoplaced)
-    (property "Reference" "R2" (at 147.32 100.33 0)
-      (effects (font (size 1.27 1.27)) (justify left))
-    )
-    (property "Value" "5.1k" (at 147.32 102.87 0)
-      (effects (font (size 1.27 1.27)) (justify left))
-    )
-    (property "Footprint" "Resistor_SMD:R_0603_1608Metric" (at 143.002 101.6 90)
-      (effects (font (size 1.27 1.27)) hide)
-    )
-    (property "Datasheet" "~" (at 144.78 101.6 0)
-      (effects (font (size 1.27 1.27)) hide)
-    )
-    (property "DigiKey" "311-5.10KHRCT-ND" (at 144.78 101.6 0)
-      (effects (font (size 1.27 1.27)) hide)
-    )
+  (symbol (lib_id "Device:R") (at 137.16 101.6 0) (unit 1)
+    (in_bom yes) (on_board yes) (dnp no) (fields_autoplaced)
+    (property "Reference" "R2" (at 139.7 100.33 0)
+      (effects (font (size 1.27 1.27)) (justify left))
+    )
+    (property "Value" "5.1k" (at 139.7 102.87 0)
+      (effects (font (size 1.27 1.27)) (justify left))
+    )
+    (property "Footprint" "Resistor_SMD:R_0603_1608Metric" (at 135.382 101.6 90)
+      (effects (font (size 1.27 1.27)) hide)
+    )
+    (property "Datasheet" "~" (at 137.16 101.6 0)
+      (effects (font (size 1.27 1.27)) hide)
+    )
+    (property "DigiKey" "311-5.10KHRCT-ND" (at 137.16 101.6 0)
+      (effects (font (size 1.27 1.27)) hide)
+    )

Commit message: Rev 2
Connections:
- net D+: now also J1.A6 (D+)
- net D-: now also J1.A7 (D-)
- no-connect marks 2 -> 0
Changed lines of the file:
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@@
   (junction (at 105.41 116.84) (diameter 0) (color 0 0 0 0)
   )
-  (no_connect (at 128.27 91.44))
-  (no_connect (at 128.27 96.52))
   (wire (pts (xy 144.78 107.95) (xy 144.78 105.41))
     (stroke (width 0) (type default))
@@
       (effects (font (size 1.27 1.27)) (justify left) hide)
     )
+  )
+  (global_label "D-" (shape input) (at 128.27 91.44 0) (fields_autoplaced)
+    (effects (font (size 1.27 1.27)) (justify left))
+    (property "Intersheetrefs" "${INTERSHEET_REFS}" (at 134.0976 91.44 0)
+      (effects (font (size 1.27 1.27)) (justify left) hide)
+    )
+  )
+  (global_label "D+" (shape input) (at 128.27 96.52 0) (fields_autoplaced)
+    (effects (font (size 1.27 1.27)) (justify left))
+    (property "Intersheetrefs" "${INTERSHEET_REFS}" (at 134.0976 96.52 0)
+      (effects (font (size 1.27 1.27)) (justify left) hide)
+    )
