File: Board/ND68.kicad_pcb (KiCad board)
At the start: 2 copper layers, 66.6 x 40.3 mm, 39 parts, among them J1 USB_C_Receptacle_USB2.0_14P, J2 Conn_01x03_Pin, U1 NCP1117-3.3_SOT223, U2 RP2040, Y1 Crystal_GND24

Commit message: Rev 2
Parts:
- added C18: 100n, Capacitor_SMD:C_0201_0603Metric, B.Cu at (173.8, 90.9)
- added C19: 100n, Capacitor_SMD:C_0201_0603Metric, B.Cu at (188.6, 88.9)
- added C20: 100n, Capacitor_SMD:C_0201_0603Metric, B.Cu at (172.2, 108.3)
- added C21: 100n, Capacitor_SMD:C_0201_0603Metric, B.Cu at (193.0, 107.6)
- added Q1: BSS138, Package_TO_SOT_SMD:SOT-23-3, B.Cu at (161.3, 91.4)
- added R7: 10k, Resistor_SMD:R_0402_1005Metric, B.Cu at (157.2, 90.5)
- added R8: 10k, Resistor_SMD:R_0402_1005Metric, B.Cu at (157.2, 86.5)
- added R9: 470, Resistor_SMD:R_0201_0603Metric, B.Cu at (155.1, 101.6)
- J2: footprint Connector_PinHeader_2.00mm:PinHeader_1x03_P2.00mm_Vertical -> Connector_PinHeader_2.54mm:PinHeader_1x03_P2.54mm_Vertical
- moved R3 7.70 mm to (135.8, 96.6)
- moved C15 2.74 mm to (144.5, 104.8), turned to 180 degrees
- moved R4 2.66 mm to (146.1, 105.3)
- moved C17 2.21 mm to (139.7, 104.0)
- moved C16 2.11 mm to (147.6, 106.0), turned to 180 degrees
- moved Y1 1.60 mm to (146.1, 108.7)
- moved J2 0.81 mm to (156.2, 108.7)
- moved C12 0.53 mm to (150.4, 106.1)
- moved C4 0.15 mm to (150.3, 104.8)
- turned SW5 to 90 degrees
Connections:
- J1 pad A6: unconnected-(J1-D+-PadA6) -> D+
- J1 pad A7: unconnected-(J1-D--PadA7) -> D-
- U2 pad 32: DIN -> Net-(U2-GPIO21)
Routing:
- net GND: track 100.1 -> 134.6 mm, vias 22 -> 40
- net VBUS: track 127.1 -> 151.1 mm, vias 1 -> 5
- net Net-(SW2-DOUT): track 65.1 -> 43.3 mm
- net Net-(Q1-S): track 0.00 -> 18.7 mm, vias 0 -> 2
- net +3.3V: track 61.6 -> 80.3 mm, vias 2 -> 6
- net DIN: track 25.3 -> 16.9 mm, vias 1 -> 0
- net QSPI_SS: track 27.2 -> 19.9 mm
- net C1: track 67.6 -> 72.2 mm
- net Net-(U2-GPIO21): track 0.00 -> 4.15 mm, vias 0 -> 1
- net R1: track 34.0 -> 37.7 mm, vias 1 -> 2
- net D+: track 14.8 -> 17.3 mm
- net C0: track 47.2 -> 49.6 mm, vias 2 -> 3
- net XIN: track 8.01 -> 10.2 mm
- net R0: track 38.2 -> 40.1 mm, vias 1 -> 2
- net Net-(R3-Pad1): track 4.53 -> 2.69 mm
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- added copper zone on F.Cu, net GND
Other:
- board text added: "ND68 MKL PROTO REV 2"
- board text removed: "ND68 MKL PROTO"

Commit message: MKL Rev 2 final
Parts:
- R1, R2: footprint Resistor_SMD:R_0603_1608Metric -> Resistor_SMD:R_0201_0603Metric
Changed lines of the file:
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@@
     )
   )
-  (footprint "Resistor_SMD:R_0603_1608Metric" (layer "F.Cu")
+  (footprint "Resistor_SMD:R_0201_0603Metric" (layer "F.Cu")
     (at 150.705 81.55 -90)
-    (descr "Resistor SMD 0603 (1608 Metric), square (rectangular) end terminal, IPC_7351 nominal, (Body size source: IPC-SM-782 page 72, https://www.pcb-3d.com/wordpress/wp-content/uploads/ipc-sm-782a_amendment_1_and_2.pdf), generated with kicad-footprint-generator")
+    (descr "Resistor SMD 0201 (0603 Metric), square (rectangular) end terminal, IPC_7351 nominal, (Body size source: https://www.vishay.com/docs/20052/crcw0201e3.pdf), generated with kicad-footprint-generator")
     (tags "resistor")
     (property "DigiKey" "311-5.10KHRCT-ND")
@@
     (property "ki_keywords" "R res resistor")
     (attr smd)
-    (fp_text reference "R1" (at 0 -1.43 90) (layer "F.SilkS")
-        (effects (font (size 1 1) (thickness 0.15)))
-    )
-    (fp_text value "5.1k" (at 0 1.43 90) (layer "F.Fab") hide
-        (effects (font (size 1 1) (thickness 0.15)))
-    )
-    (fp_text user "${REFERENCE}" (at 0 0 90) (layer "F.Fab")
-        (effects (font (size 0.4 0.4) (thickness 0.06)))
-    )
-    (fp_line (start -0.237258 -0.5225) (end 0.237258 -0.5225)
-      (stroke (width 0.12) (type solid)) (layer "F.SilkS"))
-    (fp_line (start -0.237258 0.5225) (end 0.237258 0.5225)
-      (stroke (width 0.12) (type solid)) (layer "F.SilkS"))
-    (fp_line (start -1.48 -0.73) (end 1.48 -0.73)
-      (stroke (width 0.05) (type solid)) (layer "F.CrtYd"))
-    (fp_line (start -1.48 0.73) (end -1.48 -0.73)
-      (stroke (width 0.05) (type solid)) (layer "F.CrtYd"))
-    (fp_line (start 1.48 -0.73) (end 1.48 0.73)
-      (stroke (width 0.05) (type solid)) (layer "F.CrtYd"))
-    (fp_line (start 1.48 0.73) (end -1.48 0.73)
-      (stroke (width 0.05) (type solid)) (layer "F.CrtYd"))
-    (fp_line (start -0.8 -0.4125) (end 0.8 -0.4125)
-      (stroke (width 0.1) (type solid)) (layer "F.Fab"))
-    (fp_line (start -0.8 0.4125) (end -0.8 -0.4125)
-      (stroke (width 0.1) (type solid)) (layer "F.Fab"))
-    (fp_line (start 0.8 -0.4125) (end 0.8 0.4125)
-      (stroke (width 0.1) (type solid)) (layer "F.Fab"))
-    (fp_line (start 0.8 0.4125) (end -0.8 0.4125)
-      (stroke (width 0.1) (type solid)) (layer "F.Fab"))
-    (pad "1" smd roundrect (at -0.825 0 270) (size 0.8 0.95) (layers "F.Cu" "F.Paste" "F.Mask") (roundrect_rratio 0.25)
+    (fp_text reference "R1" (at 0 -1.05 -90) (layer "F.SilkS")
+        (effects (font (size 1 1) (thickness 0.15)))
+    )
+    (fp_text value "5.1k" (at 0 1.05 -90) (layer "F.Fab")
+        (effects (font (size 1 1) (thickness 0.15)))
+    )
+    (fp_text user "${REFERENCE}" (at 0 -0.68 -90) (layer "F.Fab")
+        (effects (font (size 0.25 0.25) (thickness 0.04)))
+    )
+    (fp_line (start -0.7 -0.35) (end 0.7 -0.35)
+      (stroke (width 0.05) (type solid)) (layer "F.CrtYd"))
+    (fp_line (start -0.7 0.35) (end -0.7 -0.35)
+      (stroke (width 0.05) (type solid)) (layer "F.CrtYd"))
+    (fp_line (start 0.7 -0.35) (end 0.7 0.35)
+      (stroke (width 0.05) (type solid)) (layer "F.CrtYd"))
+    (fp_line (start 0.7 0.35) (end -0.7 0.35)
+      (stroke (width 0.05) (type solid)) (layer "F.CrtYd"))
+    (fp_line (start -0.3 -0.15) (end 0.3 -0.15)
+      (stroke (width 0.1) (type solid)) (layer "F.Fab"))
+    (fp_line (start -0.3 0.15) (end -0.3 -0.15)
+      (stroke (width 0.1) (type solid)) (layer "F.Fab"))
+    (fp_line (start 0.3 -0.15) (end 0.3 0.15)
+      (stroke (width 0.1) (type solid)) (layer "F.Fab"))
+    (fp_line (start 0.3 0.15) (end -0.3 0.15)
+      (stroke (width 0.1) (type solid)) (layer "F.Fab"))
+    (pad "" smd roundrect (at -0.345 0 270) (size 0.318 0.36) (layers "F.Paste") (roundrect_rratio 0.25))
+    (pad "" smd roundrect (at 0.345 0 270) (size 0.318 0.36) (layers "F.Paste") (roundrect_rratio 0.25))
+    (pad "1" smd roundrect (at -0.32 0 270) (size 0.46 0.4) (layers "F.Cu" "F.Mask") (roundrect_rratio 0.25)
       (net 13 "Net-(J1-CC1)") (pintype "passive"))
-    (pad "2" smd roundrect (at 0.825 0 270) (size 0.8 0.95) (layers "F.Cu" "F.Paste" "F.Mask") (roundrect_rratio 0.25)
+    (pad "2" smd roundrect (at 0.32 0 270) (size 0.46 0.4) (layers "F.Cu" "F.Mask") (roundrect_rratio 0.25)
       (net 2 "GND") (pintype "passive"))
-    (model "${KICAD6_3DMODEL_DIR}/Resistor_SMD.3dshapes/R_0603_1608Metric.wrl"
+    (model "${KICAD6_3DMODEL_DIR}/Resistor_SMD.3dshapes/R_0201_0603Metric.wrl"
       (offset (xyz 0 0 0))
       (scale (xyz 1 1 1))
@@
     )
   )
-  (footprint "Resistor_SMD:R_0603_1608Metric" (layer "F.Cu")
+  (footprint "Resistor_SMD:R_0201_0603Metric" (layer "F.Cu")
     (at 146.73625 81.55 -90)
-    (descr "Resistor SMD 0603 (1608 Metric), square (rectangular) end terminal, IPC_7351 nominal, (Body size source: IPC-SM-782 page 72, https://www.pcb-3d.com/wordpress/wp-content/uploads/ipc-sm-782a_amendment_1_and_2.pdf), generated with kicad-footprint-generator")
+    (descr "Resistor SMD 0201 (0603 Metric), square (rectangular) end terminal, IPC_7351 nominal, (Body size source: https://www.vishay.com/docs/20052/crcw0201e3.pdf), generated with kicad-footprint-generator")
     (tags "resistor")
     (property "DigiKey" "311-5.10KHRCT-ND")
@@
     (property "ki_keywords" "R res resistor")
     (attr smd)
-    (fp_text reference "R2" (at 0 1.45875 90) (layer "F.SilkS")
-        (effects (font (size 1 1) (thickness 0.15)))
-    )
-    (fp_text value "5.1k" (at 0 1.43 90) (layer "F.Fab") hide
-        (effects (font (size 1 1) (thickness 0.15)))
-    )
-    (fp_text user "${REFERENCE}" (at 0 0 90) (layer "F.Fab")
-        (effects (font (size 0.4 0.4) (thickness 0.06)))
-    )
-    (fp_line (start -0.237258 -0.5225) (end 0.237258 -0.5225)
-      (stroke (width 0.12) (type solid)) (layer "F.SilkS"))
-    (fp_line (start -0.237258 0.5225) (end 0.237258 0.5225)
-      (stroke (width 0.12) (type solid)) (layer "F.SilkS"))
-    (fp_line (start -1.48 -0.73) (end 1.48 -0.73)
-      (stroke (width 0.05) (type solid)) (layer "F.CrtYd"))
-    (fp_line (start -1.48 0.73) (end -1.48 -0.73)
-      (stroke (width 0.05) (type solid)) (layer "F.CrtYd"))
-    (fp_line (start 1.48 -0.73) (end 1.48 0.73)
-      (stroke (width 0.05) (type solid)) (layer "F.CrtYd"))
-    (fp_line (start 1.48 0.73) (end -1.48 0.73)
-      (stroke (width 0.05) (type solid)) (layer "F.CrtYd"))
-    (fp_line (start -0.8 -0.4125) (end 0.8 -0.4125)
-      (stroke (width 0.1) (type solid)) (layer "F.Fab"))
-    (fp_line (start -0.8 0.4125) (end -0.8 -0.4125)
-      (stroke (width 0.1) (type solid)) (layer "F.Fab"))
-    (fp_line (start 0.8 -0.4125) (end 0.8 0.4125)
-      (stroke (width 0.1) (type solid)) (layer "F.Fab"))
-    (fp_line (start 0.8 0.4125) (end -0.8 0.4125)
-      (stroke (width 0.1) (type solid)) (layer "F.Fab"))
-    (pad "1" smd roundrect (at -0.825 0 270) (size 0.8 0.95) (layers "F.Cu" "F.Paste" "F.Mask") (roundrect_rratio 0.25)
+    (fp_text reference "R2" (at 0 -1.05 -90) (layer "F.SilkS")
+        (effects (font (size 1 1) (thickness 0.15)))
+    )
+    (fp_text value "5.1k" (at 0 1.05 -90) (layer "F.Fab")
+        (effects (font (size 1 1) (thickness 0.15)))
+    )
+    (fp_text user "${REFERENCE}" (at 0 -0.68 -90) (layer "F.Fab")
+        (effects (font (size 0.25 0.25) (thickness 0.04)))
+    )
+    (fp_line (start -0.7 -0.35) (end 0.7 -0.35)
+      (stroke (width 0.05) (type solid)) (layer "F.CrtYd"))
+    (fp_line (start -0.7 0.35) (end -0.7 -0.35)
+      (stroke (width 0.05) (type solid)) (layer "F.CrtYd"))
+    (fp_line (start 0.7 -0.35) (end 0.7 0.35)
+      (stroke (width 0.05) (type solid)) (layer "F.CrtYd"))
+    (fp_line (start 0.7 0.35) (end -0.7 0.35)
+      (stroke (width 0.05) (type solid)) (layer "F.CrtYd"))
+    (fp_line (start -0.3 -0.15) (end 0.3 -0.15)
+      (stroke (width 0.1) (type solid)) (layer "F.Fab"))
+    (fp_line (start -0.3 0.15) (end -0.3 -0.15)
+      (stroke (width 0.1) (type solid)) (layer "F.Fab"))
+    (fp_line (start 0.3 -0.15) (end 0.3 0.15)
+      (stroke (width 0.1) (type solid)) (layer "F.Fab"))
+    (fp_line (start 0.3 0.15) (end -0.3 0.15)
+      (stroke (width 0.1) (type solid)) (layer "F.Fab"))
+    (pad "" smd roundrect (at -0.345 0 270) (size 0.318 0.36) (layers "F.Paste") (roundrect_rratio 0.25))
+    (pad "" smd roundrect (at 0.345 0 270) (size 0.318 0.36) (layers "F.Paste") (roundrect_rratio 0.25))
+    (pad "1" smd roundrect (at -0.32 0 270) (size 0.46 0.4) (layers "F.Cu" "F.Mask") (roundrect_rratio 0.25)
       (net 14 "Net-(J1-CC2)") (pintype "passive"))
-    (pad "2" smd roundrect (at 0.825 0 270) (size 0.8 0.95) (layers "F.Cu" "F.Paste" "F.Mask") (roundrect_rratio 0.25)
+    (pad "2" smd roundrect (at 0.32 0 270) (size 0.46 0.4) (layers "F.Cu" "F.Mask") (roundrect_rratio 0.25)
       (net 2 "GND") (pintype "passive"))
-    (model "${KICAD6_3DMODEL_DIR}/Resistor_SMD.3dshapes/R_0603_1608Metric.wrl"
+    (model "${KICAD6_3DMODEL_DIR}/Resistor_SMD.3dshapes/R_0201_0603Metric.wrl"
       (offset (xyz 0 0 0))
       (scale (xyz 1 1 1))

Commit message: Starting from scratch
Parts:
- removed G***: LOGO, ND68:troll
- removed Q1: BSS138, Package_TO_SOT_SMD:SOT-23-3
- added C22: 100n, Capacitor_SMD:C_0603_1608Metric, F.Cu at (502.8, 4.75)
- added C23: 100n, Capacitor_SMD:C_0603_1608Metric, F.Cu at (502.8, 7.26)
- added C24: 100n, Capacitor_SMD:C_0603_1608Metric, F.Cu at (502.8, 9.78)
- added C25: 100n, Capacitor_SMD:C_0603_1608Metric, F.Cu at (502.8, 12.3)
- added C26: 100n, Capacitor_SMD:C_0603_1608Metric, F.Cu at (502.8, 14.8)
- added C27: 100n, Capacitor_SMD:C_0603_1608Metric, F.Cu at (502.8, 17.3)
- added C28: 100n, Capacitor_SMD:C_0603_1608Metric, F.Cu at (506.8, -5.29)
- added C29: 100n, Capacitor_SMD:C_0603_1608Metric, F.Cu at (506.8, -2.77)
- added C30: 100n, Capacitor_SMD:C_0603_1608Metric, F.Cu at (506.8, -0.27)
- added C31: 100n, Capacitor_SMD:C_0603_1608Metric, F.Cu at (506.8, 2.25)
- added C32: 100n, Capacitor_SMD:C_0603_1608Metric, F.Cu at (506.8, 4.75)
- added C33: 100n, Capacitor_SMD:C_0603_1608Metric, F.Cu at (506.8, 7.26)
- added C34: 100n, Capacitor_SMD:C_0603_1608Metric, F.Cu at (506.8, 9.78)
- added C35: 100n, Capacitor_SMD:C_0603_1608Metric, F.Cu at (506.8, 12.3)
- added C36: 100n, Capacitor_SMD:C_0603_1608Metric, F.Cu at (506.8, 14.8)
- added C37: 100n, Capacitor_SMD:C_0603_1608Metric, F.Cu at (506.8, 17.3)
- added C38: 100n, Capacitor_SMD:C_0603_1608Metric, F.Cu at (510.8, -5.29)
- added C39: 100n, Capacitor_SMD:C_0603_1608Metric, F.Cu at (510.8, -2.77)
- added C40: 100n, Capacitor_SMD:C_0603_1608Metric, F.Cu at (510.8, -0.27)
- added C41: 100n, Capacitor_SMD:C_0603_1608Metric, F.Cu at (510.8, 2.25)
- added C42: 100n, Capacitor_SMD:C_0603_1608Metric, F.Cu at (510.8, 4.75)
- added C43: 100n, Capacitor_SMD:C_0603_1608Metric, F.Cu at (510.8, 7.26)
- added C44: 100n, Capacitor_SMD:C_0603_1608Metric, F.Cu at (510.8, 9.78)
- added C45: 100n, Capacitor_SMD:C_0603_1608Metric, F.Cu at (510.8, 12.3)
- added C46: 100n, Capacitor_SMD:C_0603_1608Metric, F.Cu at (510.8, 14.8)
- added C47: 100n, Capacitor_SMD:C_0603_1608Metric, F.Cu at (510.8, 17.3)
- added C48: 100n, Capacitor_SMD:C_0603_1608Metric, F.Cu at (514.8, -5.29)
- added C49: 100n, Capacitor_SMD:C_0603_1608Metric, F.Cu at (514.8, -2.77)
- added C50: 100n, Capacitor_SMD:C_0603_1608Metric, F.Cu at (514.8, -0.27)
- added C51: 100n, Capacitor_SMD:C_0603_1608Metric, F.Cu at (514.8, 2.25)
- added C52: 100n, Capacitor_SMD:C_0603_1608Metric, F.Cu at (514.8, 4.75)
- added C53: 100n, Capacitor_SMD:C_0603_1608Metric, F.Cu at (514.8, 7.26)
- added C54: 100n, Capacitor_SMD:C_0603_1608Metric, F.Cu at (514.8, 9.78)
- added C55: 100n, Capacitor_SMD:C_0603_1608Metric, F.Cu at (514.8, 12.3)
- added C56: 100n, Capacitor_SMD:C_0603_1608Metric, F.Cu at (514.8, 14.8)
- added C57: 100n, Capacitor_SMD:C_0603_1608Metric, F.Cu at (514.8, 17.3)
- added C58: 100n, Capacitor_SMD:C_0603_1608Metric, F.Cu at (518.8, -5.29)
- added C59: 100n, Capacitor_SMD:C_0603_1608Metric, F.Cu at (518.8, -2.77)
- added C60: 100n, Capacitor_SMD:C_0603_1608Metric, F.Cu at (518.8, -0.27)
- added C61: 100n, Capacitor_SMD:C_0603_1608Metric, F.Cu at (518.8, 2.25)
- added C62: 100n, Capacitor_SMD:C_0603_1608Metric, F.Cu at (518.8, 4.75)
- added C63: 100n, Capacitor_SMD:C_0603_1608Metric, F.Cu at (518.8, 7.26)
- added C64: 100n, Capacitor_SMD:C_0603_1608Metric, F.Cu at (518.8, 9.78)
- added C65: 100n, Capacitor_SMD:C_0603_1608Metric, F.Cu at (518.8, 12.3)
- added C66: 100n, Capacitor_SMD:C_0603_1608Metric, F.Cu at (518.8, 14.8)
- added C67: 100n, Capacitor_SMD:C_0603_1608Metric, F.Cu at (518.8, 17.3)
- added C68: 100n, Capacitor_SMD:C_0603_1608Metric, F.Cu at (522.8, -5.29)
- added C69: 100n, Capacitor_SMD:C_0603_1608Metric, F.Cu at (522.8, -2.77)
- added C70: 100n, Capacitor_SMD:C_0603_1608Metric, F.Cu at (522.8, -0.27)
- added C71: 100n, Capacitor_SMD:C_0603_1608Metric, F.Cu at (522.8, 2.25)
- added C72: 100n, Capacitor_SMD:C_0603_1608Metric, F.Cu at (522.8, 4.75)
- added C73: 100n, Capacitor_SMD:C_0603_1608Metric, F.Cu at (522.8, 7.26)
- added C74: 100n, Capacitor_SMD:C_0603_1608Metric, F.Cu at (522.8, 9.78)
- added C75: 100n, Capacitor_SMD:C_0603_1608Metric, F.Cu at (522.8, 12.3)
- added C76: 100n, Capacitor_SMD:C_0603_1608Metric, F.Cu at (522.8, 14.8)
- added C77: 100n, Capacitor_SMD:C_0603_1608Metric, F.Cu at (522.8, 17.3)
- added C78: 100n, Capacitor_SMD:C_0603_1608Metric, F.Cu at (526.8, -5.29)
- added C79: 100n, Capacitor_SMD:C_0603_1608Metric, F.Cu at (526.8, -2.77)
- added C80: 100n, Capacitor_SMD:C_0603_1608Metric, F.Cu at (526.8, -0.27)
- added C81: 100n, Capacitor_SMD:C_0603_1608Metric, F.Cu at (526.8, 2.25)
- added C82: 100n, Capacitor_SMD:C_0603_1608Metric, F.Cu at (526.8, 4.75)
- added C83: 100n, Capacitor_SMD:C_0603_1608Metric, F.Cu at (526.8, 7.26)
- added C84: 100n, Capacitor_SMD:C_0603_1608Metric, F.Cu at (526.8, 9.78)
- added C85: 100n, Capacitor_SMD:C_0603_1608Metric, F.Cu at (526.8, 12.3)
- added C86: 100n, Capacitor_SMD:C_0603_1608Metric, F.Cu at (526.8, 14.8)
- added C87: 100n, Capacitor_SMD:C_0603_1608Metric, F.Cu at (526.8, 17.3)
- added C88: 10u, Capacitor_SMD:C_0805_2012Metric, F.Cu at (503.0, 20.1)
- added C89: 10u, Capacitor_SMD:C_0805_2012Metric, F.Cu at (503.0, 23.1)
- added D10: D, Diode_SMD:D_SOD-123F, F.Cu at (498.8, 127.6)
- added D11: D, Diode_SMD:D_SOD-123F, F.Cu at (498.8, 130.9)
- added D12: D, Diode_SMD:D_SOD-123F, F.Cu at (498.8, 134.3)
- added D13: D, Diode_SMD:D_SOD-123F, F.Cu at (504.3, 97.4)
- added D14: D, Diode_SMD:D_SOD-123F, F.Cu at (504.3, 100.8)
- added D15: D, Diode_SMD:D_SOD-123F, F.Cu at (504.3, 104.1)
- added D16: D, Diode_SMD:D_SOD-123F, F.Cu at (504.3, 107.5)
- added D17: D, Diode_SMD:D_SOD-123F, F.Cu at (504.3, 110.8)
- added D18: D, Diode_SMD:D_SOD-123F, F.Cu at (504.3, 114.2)
- added D19: D, Diode_SMD:D_SOD-123F, F.Cu at (504.3, 117.5)
- added D20: D, Diode_SMD:D_SOD-123F, F.Cu at (504.3, 120.9)
- added D21: D, Diode_SMD:D_SOD-123F, F.Cu at (504.3, 124.2)
- added D22: D, Diode_SMD:D_SOD-123F, F.Cu at (504.3, 127.6)
- added D23: D, Diode_SMD:D_SOD-123F, F.Cu at (504.3, 130.9)
- added D24: D, Diode_SMD:D_SOD-123F, F.Cu at (504.3, 134.3)
- added D25: D, Diode_SMD:D_SOD-123F, F.Cu at (509.8, 97.4)
- added D26: D, Diode_SMD:D_SOD-123F, F.Cu at (509.8, 100.8)
- added D27: D, Diode_SMD:D_SOD-123F, F.Cu at (509.8, 104.1)
- added D28: D, Diode_SMD:D_SOD-123F, F.Cu at (509.8, 107.5)
- added D29: D, Diode_SMD:D_SOD-123F, F.Cu at (509.8, 110.8)
- added D30: D, Diode_SMD:D_SOD-123F, F.Cu at (509.8, 114.2)
- added D31: D, Diode_SMD:D_SOD-123F, F.Cu at (509.8, 117.5)
- added D32: D, Diode_SMD:D_SOD-123F, F.Cu at (509.8, 120.9)
- added D33: D, Diode_SMD:D_SOD-123F, F.Cu at (509.8, 124.2)
- added D34: D, Diode_SMD:D_SOD-123F, F.Cu at (509.8, 127.6)
- added D35: D, Diode_SMD:D_SOD-123F, F.Cu at (509.8, 130.9)
- added D36: D, Diode_SMD:D_SOD-123F, F.Cu at (509.8, 134.3)
- added D37: D, Diode_SMD:D_SOD-123F, F.Cu at (515.2, 97.4)
- added D38: D, Diode_SMD:D_SOD-123F, F.Cu at (515.2, 100.8)
- added D39: D, Diode_SMD:D_SOD-123F, F.Cu at (515.2, 104.1)
- added D40: D, Diode_SMD:D_SOD-123F, F.Cu at (515.2, 107.5)
- added D41: D, Diode_SMD:D_SOD-123F, F.Cu at (515.2, 110.8)
- added D42: D, Diode_SMD:D_SOD-123F, F.Cu at (515.2, 114.2)
- added D43: D, Diode_SMD:D_SOD-123F, F.Cu at (515.2, 117.5)
- added D44: D, Diode_SMD:D_SOD-123F, F.Cu at (515.2, 120.9)
- added D45: D, Diode_SMD:D_SOD-123F, F.Cu at (515.2, 124.2)
- added D46: D, Diode_SMD:D_SOD-123F, F.Cu at (515.2, 127.6)
- added D47: D, Diode_SMD:D_SOD-123F, F.Cu at (515.2, 130.9)
- added D48: D, Diode_SMD:D_SOD-123F, F.Cu at (515.2, 134.3)
- added D49: D, Diode_SMD:D_SOD-123F, F.Cu at (520.7, 97.4)
- added D5: D, Diode_SMD:D_SOD-123F, F.Cu at (498.8, 110.8)
- added D50: D, Diode_SMD:D_SOD-123F, F.Cu at (520.7, 100.8)
- added D51: D, Diode_SMD:D_SOD-123F, F.Cu at (520.7, 104.1)
- added D52: D, Diode_SMD:D_SOD-123F, F.Cu at (520.7, 107.5)
- added D53: D, Diode_SMD:D_SOD-123F, F.Cu at (520.7, 110.8)
- added D54: D, Diode_SMD:D_SOD-123F, F.Cu at (520.7, 114.2)
- added D55: D, Diode_SMD:D_SOD-123F, F.Cu at (520.7, 117.5)
- added D56: D, Diode_SMD:D_SOD-123F, F.Cu at (520.7, 120.9)
- added D57: D, Diode_SMD:D_SOD-123F, F.Cu at (520.7, 124.2)
- added D58: D, Diode_SMD:D_SOD-123F, F.Cu at (520.7, 127.6)
- added D59: D, Diode_SMD:D_SOD-123F, F.Cu at (520.7, 130.9)
- added D6: D, Diode_SMD:D_SOD-123F, F.Cu at (498.8, 114.2)
- added D60: D, Diode_SMD:D_SOD-123F, F.Cu at (520.7, 134.3)
- added D61: D, Diode_SMD:D_SOD-123F, F.Cu at (526.2, 97.4)
- added D62: D, Diode_SMD:D_SOD-123F, F.Cu at (526.2, 100.8)
- added D63: D, Diode_SMD:D_SOD-123F, F.Cu at (526.2, 104.1)
- added D64: D, Diode_SMD:D_SOD-123F, F.Cu at (526.2, 107.5)
- added D65: D, Diode_SMD:D_SOD-123F, F.Cu at (526.2, 110.8)
- added D66: D, Diode_SMD:D_SOD-123F, F.Cu at (526.2, 114.2)
- added D67: D, Diode_SMD:D_SOD-123F, F.Cu at (526.2, 117.5)
- added D68: D, Diode_SMD:D_SOD-123F, F.Cu at (526.2, 120.9)
- added D7: D, Diode_SMD:D_SOD-123F, F.Cu at (498.8, 117.5)
- added D8: D, Diode_SMD:D_SOD-123F, F.Cu at (498.8, 120.9)
- added D9: D, Diode_SMD:D_SOD-123F, F.Cu at (498.8, 124.2)
- added J3: Conn_01x05_Pin, Connector_PinHeader_2.54mm:PinHeader_1x05_P2.54mm_Vertical, F.Cu at (534.8, -4.21)
- added SW0: ~, ND68:PTS636 SM43 SMTR LFS, F.Cu at (538.1, 37.4)
- added SW10: ~, ND68:ND68-1U-HS-ARGB, F.Cu at (359.9, 3.56)
- added SW11: ~, ND68:ND68-1U-HS-ARGB, F.Cu at (359.9, 23.8)
- added SW12: ~, ND68:ND68-1U-HS-ARGB, F.Cu at (359.9, 44.0)
- added SW13: ~, ND68:ND68-1U-HS-ARGB, F.Cu at (359.9, 64.2)
- added SW14: ~, ND68:ND68-2U-HS-ARGB, F.Cu at (490.7, 166.4)
- added SW15: ~, ND68:ND68-1U-HS-ARGB, F.Cu at (359.9, 84.4)
- added SW16: ~, ND68:ND68-1.5U-HS-ARGB, F.Cu at (485.9, 3.56)
- added SW17: ~, ND68:ND68-1U-HS-ARGB, F.Cu at (359.9, 104.6)
- added SW18: ~, ND68:ND68-1U-HS-ARGB, F.Cu at (359.9, 124.8)
- added SW19: ~, ND68:ND68-1U-HS-ARGB, F.Cu at (359.9, 145.0)
- added SW20: ~, ND68:ND68-1U-HS-ARGB, F.Cu at (359.9, 165.2)
- added SW21: ~, ND68:ND68-1U-HS-ARGB, F.Cu at (380.1, 3.56)
- added SW22: ~, ND68:ND68-1U-HS-ARGB, F.Cu at (380.1, 23.8)
- added SW23: ~, ND68:ND68-1U-HS-ARGB, F.Cu at (380.1, 44.0)
- added SW24: ~, ND68:ND68-1U-HS-ARGB, F.Cu at (380.1, 64.2)
- added SW25: ~, ND68:ND68-1U-HS-ARGB, F.Cu at (380.1, 84.4)
- added SW26: ~, ND68:ND68-1U-HS-ARGB, F.Cu at (380.1, 104.6)
- added SW27: ~, ND68:ND68-1U-HS-ARGB, F.Cu at (380.1, 124.8)
- added SW28: ~, ND68:ND68-1U-HS-ARGB, F.Cu at (380.1, 145.0)
- added SW29: ~, ND68:ND68-1.5U-HS-ARGB, F.Cu at (485.9, 23.8)
- added SW30: ~, ND68:ND68-1U-HS-ARGB, F.Cu at (380.1, 165.2)
- added SW31: ~, ND68:ND68-1.5U-HS-ARGB, F.Cu at (485.9, 44.0)
- added SW32: ~, ND68:ND68-1U-HS-ARGB, F.Cu at (400.3, 3.56)
- added SW33: ~, ND68:ND68-1U-HS-ARGB, F.Cu at (400.3, 23.8)
- added SW34: ~, ND68:ND68-1U-HS-ARGB, F.Cu at (400.3, 44.0)
- added SW35: ~, ND68:ND68-1U-HS-ARGB, F.Cu at (400.3, 64.2)
- added SW36: ~, ND68:ND68-1U-HS-ARGB, F.Cu at (400.3, 84.4)
- added SW37: ~, ND68:ND68-1U-HS-ARGB, F.Cu at (400.3, 104.6)
- added SW38: ~, ND68:ND68-1U-HS-ARGB, F.Cu at (400.3, 124.8)
- added SW39: ~, ND68:ND68-1U-HS-ARGB, F.Cu at (400.3, 145.0)
- added SW40: ~, ND68:ND68-1U-HS-ARGB, F.Cu at (400.3, 165.2)
- added SW41: ~, ND68:ND68-1U-HS-ARGB, F.Cu at (420.5, 3.56)
- added SW42: ~, ND68:ND68-1U-HS-ARGB, F.Cu at (420.5, 23.8)
- added SW43: ~, ND68:ND68-2.25U-HS-ARGB, F.Cu at (493.0, 64.2)
- added SW44: ~, ND68:ND68-1U-HS-ARGB, F.Cu at (420.5, 44.0)
- added SW45: ~, ND68:ND68-2.25U-HS-ARGB, F.Cu at (493.0, 85.0)
- added SW46: ~, ND68:ND68-1U-HS-ARGB, F.Cu at (420.5, 64.2)
- added SW47: ~, ND68:ND68-1U-HS-ARGB, F.Cu at (420.5, 84.4)
- added SW48: ~, ND68:ND68-1U-HS-ARGB, F.Cu at (420.5, 104.6)
- added SW49: ~, ND68:ND68-1U-HS-ARGB, F.Cu at (420.5, 124.8)
- added SW50: ~, ND68:ND68-1U-HS-ARGB, F.Cu at (420.5, 145.0)
- added SW51: ~, ND68:ND68-1U-HS-ARGB, F.Cu at (420.5, 165.2)
- added SW52: ~, ND68:ND68-1U-HS-ARGB, F.Cu at (440.7, 3.56)
- added SW53: ~, ND68:ND68-1U-HS-ARGB, F.Cu at (440.7, 23.8)
- added SW54: ~, ND68:ND68-1U-HS-ARGB, F.Cu at (440.7, 44.0)
- added SW55: ~, ND68:ND68-1U-HS-ARGB, F.Cu at (440.7, 64.2)
- added SW56: ~, ND68:ND68-1.75U-HS-ARGB, F.Cu at (513.2, 146.1)
- added SW57: ~, ND68:ND68-1U-HS-ARGB, F.Cu at (440.7, 84.4)
- added SW58: ~, ND68:ND68-1U-HS-ARGB, F.Cu at (440.7, 104.6)
- added SW59: ~, ND68:ND68-1.25U-HS-ARGB, F.Cu at (483.5, 105.8)
- added SW6: ~, ND68:ND68-1U-HS-ARGB, F.Cu at (339.7, 104.6)
- added SW60: ~, ND68:ND68-1.25U-HS-ARGB, F.Cu at (483.5, 126.0)
- added SW61: ~, ND68:ND68-1.25U-HS-ARGB, F.Cu at (483.5, 146.2)
- added SW62: ~, ND68:ND68-6.25U-HS-ARGB, F.Cu at (389.7, 185.4)
- added SW63: ~, ND68:ND68-1U-HS-ARGB, F.Cu at (440.7, 124.8)
- added SW64: ~, ND68:ND68-1U-HS-ARGB, F.Cu at (440.7, 145.0)
- added SW65: ~, ND68:ND68-1U-HS-ARGB, F.Cu at (440.7, 165.2)
- added SW66: ~, ND68:ND68-1U-HS-ARGB, F.Cu at (460.9, 3.56)
- added SW67: ~, ND68:ND68-1U-HS-ARGB, F.Cu at (460.9, 23.8)
- added SW68: ~, ND68:ND68-1U-HS-ARGB, F.Cu at (460.9, 44.0)
- added SW7: ~, ND68:ND68-1U-HS-ARGB, F.Cu at (339.7, 124.8)
- added SW8: ~, ND68:ND68-1U-HS-ARGB, F.Cu at (339.7, 145.0)
- added SW9: ~, ND68:ND68-1U-HS-ARGB, F.Cu at (339.7, 165.2)
- added U4: ~, ND68:ND68-1U-ARGB_LED_ONLY, F.Cu at (460.9, 64.2)
- added U5: ~, ND68:ND68-1U-ARGB_LED_ONLY, F.Cu at (460.9, 84.4)
- C18, C19, C20, C21: footprint Capacitor_SMD:C_0201_0603Metric -> Capacitor_SMD:C_0603_1608Metric; moved to F.Cu
- D1, D2, D3, D4, R7, R8: moved to F.Cu
- R1, R2: footprint Resistor_SMD:R_0201_0603Metric -> Resistor_SMD:R_0603_1608Metric
- R9: footprint Resistor_SMD:R_0201_0603Metric -> Resistor_SMD:R_0603_1608Metric; moved to F.Cu
- SW5: footprint ND68:PTS636 SM43 SMTR LFS -> ND68:ND68-1U-HS-ARGB
- moved C11 419.5 mm to (547.9, -5.67), turned to 0 degrees
- moved C17 417.4 mm to (544.0, 0.21), turned to 0 degrees
- moved C10 415.4 mm to (545.5, -2.17), turned to 0 degrees
- moved C1 414.6 mm to (544.5, 26.0), turned to 0 degrees
- moved C12 412.5 mm to (547.9, -3.92)
- moved C2 412.2 mm to (544.5, 29.0), turned to 0 degrees
- moved C9 410.2 mm to (545.5, -3.92), turned to 0 degrees
- moved C8 409.8 mm to (545.5, -5.67), turned to 0 degrees
- moved R6 408.8 mm to (547.9, 6.14), turned to 0 degrees
- moved C5 408.6 mm to (543.0, -3.92), turned to 0 degrees
- moved R5 408.3 mm to (547.9, 4.16), turned to 0 degrees
- moved C4 407.9 mm to (543.0, -5.67)
- moved C3 407.8 mm to (547.7, -0.30), turned to 0 degrees
- moved C13 407.4 mm to (547.9, -2.17)
- moved C6 406.4 mm to (547.7, 1.67), turned to 0 degrees
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Connections:
- C18 pad 2: GND -> Net-(SW1-VDD)
- C19 pad 2: GND -> Net-(SW2-VDD)
- C20 pad 2: GND -> Net-(SW3-VDD)
- C21 pad 2: GND -> Net-(SW4-VDD)
- D3 pad 1: R1 -> R0
- D4 pad 1: R1 -> R0
- R9 pad 1: Net-(U2-GPIO21) -> unconnected-(R9-Pad1)
- SW1 pad 1: VBUS -> Net-(SW1-VDD)
- SW2 pad 1: VBUS -> Net-(SW2-VDD)
- SW3 pad 1: VBUS -> Net-(SW3-VDD)
- SW3 pad 6: C0 -> C2
- SW4 pad 1: VBUS -> Net-(SW4-VDD)
- SW4 pad 2: unconnected-(SW4-DOUT-Pad2) -> Net-(SW4-DOUT)
- SW4 pad 6: C1 -> C3
- SW5 pad 1: GND -> Net-(SW5-VDD)
- SW5 pad 2: Net-(R3-Pad1) -> Net-(SW5-DOUT)
- U2 pad 32: Net-(U2-GPIO21) -> unconnected-(U2-GPIO21-Pad32)
- U2 pad 34: C1 -> unconnected-(U2-GPIO22-Pad34)
- U2 pad 35: C0 -> unconnected-(U2-GPIO23-Pad35)
- U2 pad 36: R1 -> unconnected-(U2-GPIO24-Pad36)
- U2 pad 37: R0 -> unconnected-(U2-GPIO25-Pad37)
Routing:
- net VBUS: track 151.1 -> 0.00 mm, vias 5 -> 0
- net GND: track 134.6 -> 0.00 mm, vias 40 -> 0
- net +3.3V: track 80.3 -> 0.00 mm, vias 6 -> 0
- net C1: track 72.2 -> 0.00 mm, vias 1 -> 0
- net C0: track 49.6 -> 0.00 mm, vias 3 -> 0
- net Net-(SW2-DOUT): track 43.3 -> 0.00 mm, vias 2 -> 0
- net R0: track 40.1 -> 0.00 mm, vias 2 -> 0
- net R1: track 37.7 -> 0.00 mm, vias 2 -> 0
- net +1V1: track 21.4 -> 0.00 mm
- net QSPI_SS: track 19.9 -> 0.00 mm
- net Net-(Q1-S): track 18.7 -> 0.00 mm, vias 2 -> 0
- net D+: track 17.3 -> 0.00 mm
- net QSPI_SD1: track 17.0 -> 0.00 mm
- net DIN: track 16.9 -> 0.00 mm
- net D-: track 16.2 -> 0.00 mm
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- removed copper zone on F.Cu, net +3.3V
- removed copper zone on B.Cu, net GND
- removed copper zone on F.Cu, net GND
Other:
- board size 66.6 x 40.3 mm -> 3.4 x 3 mm
- board text removed: "CLK SWD"
- board text removed: "ND68 MKL PROTO REV 2"
