File: Board/ND68.kicad_pcb (KiCad board)
At the start: 2 copper layers, 303 x 94.2 mm, 244 parts, among them J1 USB_C_Receptacle_USB2.0_14P, J2 Conn_01x03_Pin, J3 Conn_01x05_Pin, U1 NCP1117-3.3_SOT223, U2 RP2040, Y1 Crystal_GND24

Commit message: Finished PCB keyboard matrix & diodes
Parts:
- C18, C19, C20, C21, C22, C23, C24, C25, C26, C27, C28, C29, C30, C31, C32, C34, C35, C48, C49, C50, C62, C76, C77, D1, D10, D11, D12, D13, D14, D15, D16, D17, D18, D19, D2, D20, D21, D22, D23, D24, D25, D26, D27, D28, D29, D3, D30, D31, D32, D33, D34, D35, D36, D37, D38, D39, D4, D40, D41, D42, D43, D44, D45, D46, D47, D48, D49, D5, D50, D51, D52, D53, D54, D55, D56, D57, D58, D59, D6, D60, D61, D62, D63, D64, D65, D66, D67, D68, D7, D8, D9: moved to B.Cu
- moved D59 518.3 mm to (19.8, -2.38), turned to 90 degrees
- moved D1 512.5 mm to (17.5, -78.6), turned to 90 degrees
- moved D31 510.2 mm to (24.6, -40.5), turned to 90 degrees
- moved D16 510.1 mm to (22.2, -59.5), turned to 90 degrees
- moved C76 508.4 mm to (15.1, -11.9), turned to 180 degrees
- moved D45 507.2 mm to (29.4, -21.4), turned to 90 degrees
- moved C48 497.0 mm to (19.8, -50.0), turned to 180 degrees
- moved D60 496.3 mm to (43.7, -2.38), turned to 90 degrees
- moved D2 495.8 mm to (36.5, -78.6), turned to 90 degrees
- moved C62 495.5 mm to (24.6, -31.0), turned to 180 degrees
- moved D17 488.9 mm to (46.0, -59.5), turned to 90 degrees
- moved D32 486.5 mm to (50.8, -40.5), turned to 90 degrees
- moved C77 484.8 mm to (38.9, -11.9), turned to 180 degrees
- moved D3 479.4 mm to (55.6, -78.6), turned to 90 degrees
- moved D46 478.7 mm to (60.3, -21.4), turned to 90 degrees
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Connections:
- SW14 pad 5: (no net) -> Net-(D14-A)
- SW14 pad 6: (no net) -> C13
- SW16 pad 5: (no net) -> Net-(D16-A)
- SW16 pad 6: (no net) -> C0
- SW29 pad 5: (no net) -> Net-(D29-A)
- SW29 pad 6: (no net) -> C13
- SW31 pad 5: (no net) -> Net-(D31-A)
- SW31 pad 6: (no net) -> C0
- SW43 pad 5: (no net) -> Net-(D43-A)
- SW43 pad 6: (no net) -> C12
- SW45 pad 5: (no net) -> Net-(D45-A)
- SW45 pad 6: (no net) -> C0
- SW56 pad 5: (no net) -> Net-(D56-A)
- SW56 pad 6: (no net) -> C11
- SW59 pad 5: (no net) -> Net-(D59-A)
- SW59 pad 6: (no net) -> C0
- SW60 pad 5: (no net) -> Net-(D60-A)
- SW60 pad 6: (no net) -> C1
- SW61 pad 5: (no net) -> Net-(D61-A)
- SW61 pad 6: (no net) -> C2
- SW62 pad 5: (no net) -> Net-(D62-A)
- SW62 pad 6: (no net) -> C3
Routing:
- net C8: track 0.00 -> 174.6 mm, vias 0 -> 8
- net C9: track 0.00 -> 174.5 mm, vias 0 -> 8
- net C6: track 0.00 -> 173.6 mm, vias 0 -> 10
- net C5: track 0.00 -> 172.3 mm, vias 0 -> 8
- net C7: track 0.00 -> 172.1 mm, vias 0 -> 12
- net C4: track 0.00 -> 168.4 mm, vias 0 -> 8
- net C3: track 0.00 -> 121.7 mm, vias 0 -> 8
- net C1: track 0.00 -> 100.8 mm, vias 0 -> 8
- net C2: track 0.00 -> 96.4 mm, vias 0 -> 8
- net C0: track 0.00 -> 90.4 mm
- net C13: track 0.00 -> 77.7 mm, vias 0 -> 6
- net C12: track 0.00 -> 74.0 mm, vias 0 -> 6
- net C11: track 0.00 -> 71.3 mm, vias 0 -> 6
- net C10: track 0.00 -> 67.0 mm, vias 0 -> 6
- net C14: track 0.00 -> 20.1 mm, vias 0 -> 2
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Other:
- board size 303 x 94.2 mm -> 304.8 x 105.6 mm
- board text added: "311-1088-2-ND*68"
- board text added: "4878-1N4148WCT-ND*68"
- board text added: "ND68 TKL Proto REV 1"

Commit message: Wire capacitors and wire up diode matrix
Parts:
- C33, C36, C37, C38, C39, C40, C41, C42, C43, C44, C45, C46, C47, C51, C52, C53, C54, C55, C56, C57, C58, C59, C60, C61, C63, C64, C65, C66, C67, C68, C69, C70, C71, C72, C73, C74, C75, C78, C79, C80, C81, C82, C83, C84, C85, C86, C87, C88, C89: moved to B.Cu
- moved C33 495.2 mm to (17.5, -69.1), turned to 180 degrees
- moved C63 464.8 mm to (55.6, -31.0), turned to 180 degrees
- moved C78 464.1 mm to (62.7, -11.9), turned to 180 degrees
- moved C64 446.1 mm to (74.6, -31.0), turned to 180 degrees
- moved C88 438.9 mm to (69.7, -50.0)
- moved C36 435.5 mm to (79.4, -69.1), turned to 180 degrees
- moved C51 433.8 mm to (84.1, -50.0), turned to 180 degrees
- moved C86 428.7 mm to (98.4, -1.59), turned to 180 degrees
- moved C65 427.3 mm to (93.6, -31.0), turned to 180 degrees
- moved C37 417.4 mm to (98.4, -69.1), turned to 180 degrees
- moved C52 415.2 mm to (103.2, -50.0), turned to 180 degrees
- moved C66 408.7 mm to (112.7, -31.0), turned to 180 degrees
- moved C38 398.0 mm to (117.5, -69.1), turned to 180 degrees
- moved C53 396.7 mm to (122.2, -50.0), turned to 180 degrees
- moved C79 392.8 mm to (134.1, -11.9), turned to 180 degrees
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Routing:
- net R0: track 0.00 -> 291.9 mm, vias 0 -> 28
- net R4: track 0.00 -> 287.6 mm
- net R2: track 0.00 -> 284.7 mm, vias 0 -> 26
- net R3: track 0.00 -> 283.2 mm, vias 0 -> 18
- net R1: track 0.00 -> 283.0 mm, vias 0 -> 26
- net Net-(D53-A): track 0.00 -> 3.56 mm
- net Net-(U5-VDD): track 0.00 -> 2.29 mm
- net Net-(U4-VDD): track 0.00 -> 2.29 mm
- net Net-(SW62-VDD): track 0.00 -> 1.89 mm
- net Net-(SW66-VDD): track 0.00 -> 1.89 mm
- net Net-(SW65-VDD): track 0.00 -> 1.89 mm
- net Net-(SW56-VDD): track 0.00 -> 1.89 mm
- net Net-(SW54-VDD): track 0.00 -> 1.89 mm
- net Net-(SW27-VDD): track 0.00 -> 1.89 mm
- net Net-(SW22-VDD): track 0.00 -> 1.89 mm
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