File: Board/_autosave-ND68.kicad_pcb (KiCad board)
At the start: 2 copper layers, 303 x 94.2 mm, 244 parts, among them J1 USB_C_Receptacle_USB2.0_14P, J2 Conn_01x03_Pin, J3 Conn_01x05_Pin, U1 NCP1117-3.3_SOT223, U2 RP2040, Y1 Crystal_GND24

Commit message: WIP Layout, all keys placed
Changed lines of the file:
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@@
         (effects (font (size 0.8 0.8) (thickness 0.15)))
     )
-    (fp_text user "L CNRN" (at -2.794 8.7884 unlocked) (layer "F.SilkS")
+    (fp_text user "L CNRN" (at -2.794 8.7884 unlocked) (layer "F.SilkS") hide
         (effects (font (size 1 1) (thickness 0.1)) (justify left bottom))
     )
@@
         (effects (font (size 0.8 0.8) (thickness 0.15)))
     )
-    (fp_text user "L CNRN" (at -2.794 8.7884 unlocked) (layer "F.SilkS")
+    (fp_text user "L CNRN" (at -2.794 8.7884 unlocked) (layer "F.SilkS") hide
         (effects (font (size 1 1) (thickness 0.1)) (justify left bottom))
     )
